File: res/sch-v1/sch-v1.kicad_sch (KiCad schematic)
At the start: 9 parts, among them U1 WeMos_D1_mini, U2 CC56-12SURKWA

Commit message: up
Parts:
- removed R4, R5, R6, R7: 270, symbol Device:R
- removed U2: CC56-12SURKWA, Display_7Segment:CA56-12SURKWA, symbol Display_Character:CC56-12SURKWA
- added BT1: CR2032, symbol Device:Battery_Cell
- added C1, C3, C5: 100n, symbol Device:C
- added C2, C4: 10uF, symbol Device:C
- added C6: 10n, symbol Device:C
- added J1: Nixie, Connector_PinHeader_2.54mm:PinHeader_1x06_P2.54mm_Vertical, symbol Connector_Generic:Conn_01x06
- added LS1: Speaker, symbol Device:Speaker
- added PS1: Power supply, symbol Converter_ACDC:TMLM04253
- added SW1: AP On, symbol Switch:SW_Push
- added U2: AMS1117-3.3, Package_TO_SOT_SMD:SOT-223-3_TabPin2, symbol Regulator_Linear:AMS1117-3.3
- added U3: aP89341, symbol alex:aP89341
- added U4: DS1307Z+, Package_DIP:DIP-8-16_W7.62mm, symbol Timer_RTC:DS1307Z+
- added Y1: 32768, symbol Device:Crystal
- R1: value 270 -> 65k*
- R2, R3: value 270 -> 10k
Connections:
- net SEG_CR is gone; now on net +3.3V: R3.2
- net GND: now reaches U1.10 (GND)
- net GND: now also BT1.2 (-), C1.2, C2.2, C3.2, C4.2, C5.2, C6.2, J1.5 (Pin_5), PS1.3 (Common), SW1.2, U2.1 (GND), U3.11 (AVss), U3.3 (Vss), U4.4 (GND)
- net +5V: now reaches U1.9 (5V)
- net +5V: now also C1.1, C2.1, J1.4 (Pin_4), PS1.2 (Vout1), U2.3 (VI)
- net DIG_1 renamed AP_CS
- net AP_CS: now also U3.19 (S1)
- net DIG_2 renamed BTN_AP
- net BTN_AP: now also C5.1, SW1.1
- net DIG_3 renamed STROBE
- net STROBE: now also J1.2 (Pin_2)
- net DIG_4 renamed SDATA
- net SDATA: now also J1.3 (Pin_3), U3.21 (S3)
- net SEG_A: no longer names the net of U1.15 (RX)
- net SEG_A: no longer R1.1
- net SEG_AR: no longer names the net of R1.2
- net SEG_AR: now also U3.9 (OSC)
- net SEG_B: no longer names the net of U1.11 (D4)
- net SEG_B: no longer R2.1
- net SEG_BR renamed +3.3V
- net +3.3V: now also R1.1, C3.1, C4.1, U2.2 (VO), U3.6 (Vdd), U3.7 (AVdd), U4.8 (VCC)
- net SEG_C: no longer names the net of U1.16 (TX)
- net SEG_C: no longer R3.1
- net SEG_D renamed SDA
- net SDA: now also R3.1, U4.5 (SDA)
- net SEG_E renamed SCL
- net SCL: now also R2.1, U4.6 (SCL)
- net SEG_F renamed SHIFT
- net SHIFT: now also J1.1 (Pin_1), U3.20 (S2)
- net SEG_G: no longer names the net of U1.12 (D3)
- new net: BT1.1 (+), U4.3 (VBAT)
- new net: C6.1, U3.15 (RST)
- new net: U4.2 (X2), Y1.1
- new net: U4.1 (X1), Y1.2
- new net +180V: J1.6 (Pin_6), PS1.4 (Vout2)
- new net sp1: LS1.1, U3.4 (VOUT1)
- new net sp2: LS1.2, U3.5 (VOUT2)
Other:
- moved on the sheet: U1
